Commit message: worked on restaurant chairs

File: simulation_ws/src/cam_pack/urdf/factory_fisheye.xacro (robot description, xacro)
@@ -66,22 +66,23 @@
         <static>true</static>
     </gazebo>
- <link name="link2">
-        <visual>
-        <origin xyz="0 0 0" rpy="0 0 0"/>  created at 31 meters above just to have space to work with
-        <geometry>
-            <box size="0.5 0.5 0.1"/>
-        </geometry>
-        <material name = "blue"/>
-        </visual>
-    </link>
-    <gazebo reference="link2">
-        <material>Gazebo/Blue</material>
-        <static>true</static>
-    </gazebo>
-      <joint name="join2" type="fixed">
-        <origin xyz="${1*cam_separation} ${-1*cam_separation} 0" rpy="0 0 0"/>
-        <parent link="base_link"/>
-        <child link="link2"/>
-    </joint>
+<!-- <link name="link2">-->
+<!--        <visual>-->
+<!--        <origin xyz="0 0 0" rpy="0 0 0"/>  created at 31 meters above just to have space to work with-->
+<!--        <geometry>-->
+<!--            <box size="0.5 0.5 0.1"/>-->
+<!--        </geometry>-->
+<!--        <material name = "blue"/>-->
+<!--        </visual>-->
+<!--    </link>-->
+<!--     -->
+<!--    <gazebo reference="link2">-->
+<!--        <material>Gazebo/Blue</material>-->
+<!--        <static>true</static>-->
+<!--    </gazebo>-->
+<!--      <joint name="join2" type="fixed">-->
+<!--        <origin xyz="${1*cam_separation} ${-1*cam_separation} 0" rpy="0 0 0"/> -->
+<!--        <parent link="base_link"/>-->
+<!--        <child link="link2"/>-->
+<!--    </joint>-->
 <!-- <link name="link1">
         <visual>
