Commit message: Adding additional scripts

File: simulation_ws/src/cam_pack/urdf/warehouse.xacro (robot description, xacro)
@@ -1,9 +1,9 @@
- <?xml version="1.0" ?>
-<robot name="factory_cam" xmlns:xacro="http://www.ros.org/wiki/xacro" >
-<xacro:include filename = "$(find cam_pack)/urdf/factory_fisheye_cam.plugins.xacro"/>
-<xacro:property name="height_off_ground" value="10" />
+<?xml version="1.0" ?>
+<robot name="warehouse" xmlns:xacro="http://www.ros.org/wiki/xacro" >
+<xacro:include filename = "$(find cam_pack)/urdf/warehouse.plugins.xacro"/>
+<xacro:property name="height_off_ground" value="7" />
 <xacro:property name="height_off_ground_offset" value="0.2" />
 <xacro:property name="cam_separation" value="10" />
-<xacro:property name="cam_box_size" value="0.07" />
+<xacro:property name="cam_box_size" value="0.1" />
 <xacro:property name="cam_mass" value="0.25" />
 <xacro:property name="cam_z_joint_height" value="${height_off_ground - height_off_ground_offset}" />
@@ -15,7 +15,7 @@
 <xacro:property name="ceiling_inertia_yy" value="337.66666666666674" />
 <xacro:property name="ceiling_inertia_zz" value="487.50000000000006" />
-<xacro:property name="ceiling_width" value="30" />
-<xacro:property name="ceiling_length" value="50" />
-<xacro:property name="ceiling_thickness" value="0.5" />
+<xacro:property name="ceiling_width" value="0.001" />
+<xacro:property name="ceiling_length" value="0.001" />
+<xacro:property name="ceiling_thickness" value="0.001" />
     <!-- Specify material colors here -->
     <material name="blue">
@@ -31,5 +31,5 @@
     <gazebo>
         <plugin name="gazebo_ros_control" filename="libgazebo_ros_control.so">
-            <robotNamespace>/factory_cam</robotNamespace> This robot name is the same as robot name at the top
+            <robotNamespace>/warehouse</robotNamespace> This robot name is the same as robot name at the top
         </plugin>
     </gazebo>
@@ -59,22 +59,9 @@
     only for URDF coloring
     <gazebo reference="base_link">
-        <!-- <gravity>false</gravity> -->
+<!--        <gravity>false</gravity>-->
         <turnGravityOff>true</turnGravityOff>
         <mu1>10.0</mu1>
         <mu2>10.0</mu2>
         <material>Gazebo/DarkGrey</material>
-        <static>true</static>
-    </gazebo>
-     <link name="bb">
-        <visual>
-        <origin xyz="0 0 0" rpy="0 0 0"/>  created at 31 meters above just to have space to work with
-        <geometry>
-            <box size="4 4 .01"/>
-        </geometry>
-        <material name = "blue"/>
-        </visual>
-    </link>
-    <gazebo reference="bb">
-        <material>Gazebo/Blue</material>
         <static>true</static>
     </gazebo>
@@ -103,5 +90,5 @@
     </link>
     <gazebo reference="camera_link_1">
-        <!-- <gravity>false</gravity> -->
+<!--        <gravity>false</gravity>-->
         <turnGravityOff>true</turnGravityOff>
         <mu1>10.0</mu1>
@@ -132,5 +119,5 @@
     </link>
     <gazebo reference="camera_link_2">
-        <!-- <gravity>false</gravity> -->
+<!--        <gravity>false</gravity>-->
         <turnGravityOff>true</turnGravityOff>
         <mu1>10.0</mu1>
@@ -161,5 +148,5 @@
     </link>
     <gazebo reference="camera_link_3">
-        <!-- <gravity>false</gravity> -->
+<!--        <gravity>false</gravity>-->
         <turnGravityOff>true</turnGravityOff>
         <mu1>10.0</mu1>
@@ -190,5 +177,5 @@
     </link>
     <gazebo reference="camera_link_4">
-        <!-- <gravity>false</gravity> -->
+<!--        <gravity>false</gravity>-->
         <turnGravityOff>true</turnGravityOff>
         <mu1>10.0</mu1>
@@ -219,5 +206,5 @@
     </link>
     <gazebo reference="camera_link_5">
-        <!-- <gravity>false</gravity> -->
+<!--        <gravity>false</gravity>-->
         <turnGravityOff>true</turnGravityOff>
         <mu1>10.0</mu1>
@@ -248,5 +235,5 @@
     </link>
     <gazebo reference="camera_link_6">
-        <!-- <gravity>false</gravity> -->
+<!--        <gravity>false</gravity>-->
         <turnGravityOff>true</turnGravityOff>
         <mu1>10.0</mu1>
@@ -277,5 +264,5 @@
     </link>
     <gazebo reference="camera_link_7">
-        <!-- <gravity>false</gravity> -->
+<!--        <gravity>false</gravity>-->
         <turnGravityOff>true</turnGravityOff>
         <mu1>10.0</mu1>
@@ -306,5 +293,5 @@
     </link>
     <gazebo reference="camera_link_8">
-        <!-- <gravity>false</gravity> -->
+<!--        <gravity>false</gravity>-->
         <turnGravityOff>true</turnGravityOff>
         <mu1>10.0</mu1>
@@ -335,5 +322,5 @@
     </link>
     <gazebo reference="camera_link_9">
-        <!-- <gravity>false</gravity> -->
+<!--        <gravity>false</gravity>-->
         <turnGravityOff>true</turnGravityOff>
         <mu1>10.0</mu1>
@@ -364,5 +351,5 @@
     </link>
     <gazebo reference="camera_link_10">
-        <!-- <gravity>false</gravity> -->
+<!--        <gravity>false</gravity>-->
         <turnGravityOff>true</turnGravityOff>
         <mu1>10.0</mu1>
@@ -393,5 +380,5 @@
     </link>
     <gazebo reference="camera_link_11">
-        <!-- <gravity>false</gravity> -->
+<!--        <gravity>false</gravity>-->
         <turnGravityOff>true</turnGravityOff>
         <mu1>10.0</mu1>
@@ -422,5 +409,5 @@
     </link>
     <gazebo reference="camera_link_12">
-        <!-- <gravity>false</gravity> -->
+<!--        <gravity>false</gravity>-->
         <turnGravityOff>true</turnGravityOff>
         <mu1>10.0</mu1>
@@ -451,5 +438,5 @@
     </link>
     <gazebo reference="camera_link_13">
-        <!-- <gravity>false</gravity> -->
+<!--        <gravity>false</gravity>-->
         <turnGravityOff>true</turnGravityOff>
         <mu1>10.0</mu1>
@@ -480,5 +467,5 @@
     </link>
     <gazebo reference="camera_link_14">
-        <!-- <gravity>false</gravity> -->
+<!--        <gravity>false</gravity>-->
         <turnGravityOff>true</turnGravityOff>
         <mu1>10.0</mu1>
@@ -509,5 +496,266 @@
     </link>
     <gazebo reference="camera_link_15">
-        <!-- <gravity>false</gravity> -->
+<!--        <gravity>false</gravity>-->
+        <turnGravityOff>true</turnGravityOff>
+        <mu1>10.0</mu1>
+        <mu2>10.0</mu2>
+        <material>Gazebo/Red</material>
+        <static>true</static>
+    </gazebo>
+        <!-- Camera Link 16-->
+    <link name="camera_link_16">
+        <collision>
+        <origin xyz="0 0 0" rpy="0 0 0"/>
+        <geometry>
+            <box size="${cam_box_size} ${cam_box_size} ${cam_box_size}"/>
+        </geometry>
+        </collision>
+        <visual>
+        <origin xyz="0 0 0" rpy="0 0 0"/>
+        <geometry>
+            <box size="${cam_box_size} ${cam_box_size} ${cam_box_size}"/>
+        </geometry>
+        <material name="red"/>
+        </visual>
+        <inertial>
+        <mass value="${cam_mass}" /> This camera was estimated from the mass(weight) of a logitech camera = 0.25kg
+        <origin xyz="0 0 0" rpy="0 0 0"/> Inertia was calculated from the inertial calculator program
+        <inertia ixx="${cam_inertia_xx}" ixy="0" ixz="0" iyy="${cam_inertia_yy}" iyz="0" izz="${cam_inertia_zz}" />
+        </inertial>
+    </link>
+    <gazebo reference="camera_link_16">
+<!--        <gravity>false</gravity>-->
+        <turnGravityOff>true</turnGravityOff>
+        <mu1>10.0</mu1>
+        <mu2>10.0</mu2>
+        <material>Gazebo/Red</material>
+        <static>true</static>
+    </gazebo>
+        <!-- Camera Link 17-->
+    <link name="camera_link_17">
+        <collision>
+        <origin xyz="0 0 0" rpy="0 0 0"/>
+        <geometry>
+            <box size="${cam_box_size} ${cam_box_size} ${cam_box_size}"/>
+        </geometry>
+        </collision>
+        <visual>
+        <origin xyz="0 0 0" rpy="0 0 0"/>
+        <geometry>
+            <box size="${cam_box_size} ${cam_box_size} ${cam_box_size}"/>
+        </geometry>
+        <material name="red"/>
+        </visual>
+        <inertial>
+        <mass value="${cam_mass}" /> This camera was estimated from the mass(weight) of a logitech camera = 0.25kg
+        <origin xyz="0 0 0" rpy="0 0 0"/> Inertia was calculated from the inertial calculator program
+        <inertia ixx="${cam_inertia_xx}" ixy="0" ixz="0" iyy="${cam_inertia_yy}" iyz="0" izz="${cam_inertia_zz}" />
+        </inertial>
+    </link>
+    <gazebo reference="camera_link_17">
+<!--        <gravity>false</gravity>-->
+        <turnGravityOff>true</turnGravityOff>
+        <mu1>10.0</mu1>
+        <mu2>10.0</mu2>
+        <material>Gazebo/Red</material>
+        <static>true</static>
+    </gazebo>
+    <!-- Camera Link 18-->
+    <link name="camera_link_18">
+        <collision>
+        <origin xyz="0 0 0" rpy="0 0 0"/>
+        <geometry>
+            <box size="${cam_box_size} ${cam_box_size} ${cam_box_size}"/>
+        </geometry>
+        </collision>
+        <visual>
+        <origin xyz="0 0 0" rpy="0 0 0"/>
+        <geometry>
+            <box size="${cam_box_size} ${cam_box_size} ${cam_box_size}"/>
+        </geometry>
+        <material name="red"/>
+        </visual>
+        <inertial>
+        <mass value="${cam_mass}" /> This camera was estimated from the mass(weight) of a logitech camera = 0.25kg
+        <origin xyz="0 0 0" rpy="0 0 0"/> Inertia was calculated from the inertial calculator program
+        <inertia ixx="${cam_inertia_xx}" ixy="0" ixz="0" iyy="${cam_inertia_yy}" iyz="0" izz="${cam_inertia_zz}" />
+        </inertial>
+    </link>
+    <gazebo reference="camera_link_18">
+<!--        <gravity>false</gravity>-->
+        <turnGravityOff>true</turnGravityOff>
+        <mu1>10.0</mu1>
+        <mu2>10.0</mu2>
+        <material>Gazebo/Red</material>
+        <static>true</static>
+    </gazebo>
+        <!-- Camera Link 19-->
+    <link name="camera_link_19">
+        <collision>
+        <origin xyz="0 0 0" rpy="0 0 0"/>
+        <geometry>
+            <box size="${cam_box_size} ${cam_box_size} ${cam_box_size}"/>
+        </geometry>
+        </collision>
+        <visual>
+        <origin xyz="0 0 0" rpy="0 0 0"/>
+        <geometry>
+            <box size="${cam_box_size} ${cam_box_size} ${cam_box_size}"/>
+        </geometry>
+        <material name="red"/>
+        </visual>
+        <inertial>
+        <mass value="${cam_mass}" /> This camera was estimated from the mass(weight) of a logitech camera = 0.25kg
+        <origin xyz="0 0 0" rpy="0 0 0"/> Inertia was calculated from the inertial calculator program
+        <inertia ixx="${cam_inertia_xx}" ixy="0" ixz="0" iyy="${cam_inertia_yy}" iyz="0" izz="${cam_inertia_zz}" />
+        </inertial>
+    </link>
+    <gazebo reference="camera_link_19">
+<!--        <gravity>false</gravity>-->
+        <turnGravityOff>true</turnGravityOff>
+        <mu1>10.0</mu1>
+        <mu2>10.0</mu2>
+        <material>Gazebo/Red</material>
+        <static>true</static>
+    </gazebo>
+    <!-- Camera Link 20-->
+    <link name="camera_link_20">
+        <collision>
+        <origin xyz="0 0 0" rpy="0 0 0"/>
+        <geometry>
+            <box size="${cam_box_size} ${cam_box_size} ${cam_box_size}"/>
+        </geometry>
+        </collision>
+        <visual>
+        <origin xyz="0 0 0" rpy="0 0 0"/>
+        <geometry>
+            <box size="${cam_box_size} ${cam_box_size} ${cam_box_size}"/>
+        </geometry>
+        <material name="red"/>
+        </visual>
+        <inertial>
+        <mass value="${cam_mass}" /> This camera was estimated from the mass(weight) of a logitech camera = 0.25kg
+        <origin xyz="0 0 0" rpy="0 0 0"/> Inertia was calculated from the inertial calculator program
+        <inertia ixx="${cam_inertia_xx}" ixy="0" ixz="0" iyy="${cam_inertia_yy}" iyz="0" izz="${cam_inertia_zz}" />
+        </inertial>
+    </link>
+    <gazebo reference="camera_link_20">
+<!--        <gravity>false</gravity>-->
+        <turnGravityOff>true</turnGravityOff>
+        <mu1>10.0</mu1>
+        <mu2>10.0</mu2>
+        <material>Gazebo/Red</material>
+        <static>true</static>
+    </gazebo>
+        <!-- Camera Link 21-->
+    <link name="camera_link_21">
+        <collision>
+        <origin xyz="0 0 0" rpy="0 0 0"/>
+        <geometry>
+            <box size="${cam_box_size} ${cam_box_size} ${cam_box_size}"/>
+        </geometry>
+        </collision>
+        <visual>
+        <origin xyz="0 0 0" rpy="0 0 0"/>
+        <geometry>
+            <box size="${cam_box_size} ${cam_box_size} ${cam_box_size}"/>
+        </geometry>
+        <material name="red"/>
+        </visual>
+        <inertial>
+        <mass value="${cam_mass}" /> This camera was estimated from the mass(weight) of a logitech camera = 0.25kg
+        <origin xyz="0 0 0" rpy="0 0 0"/> Inertia was calculated from the inertial calculator program
+        <inertia ixx="${cam_inertia_xx}" ixy="0" ixz="0" iyy="${cam_inertia_yy}" iyz="0" izz="${cam_inertia_zz}" />
+        </inertial>
+    </link>
+    <gazebo reference="camera_link_21">
+<!--        <gravity>false</gravity>-->
+        <turnGravityOff>true</turnGravityOff>
+        <mu1>10.0</mu1>
+        <mu2>10.0</mu2>
+        <material>Gazebo/Red</material>
+        <static>true</static>
+    </gazebo>
+        <!-- Camera Link 22-->
+    <link name="camera_link_22">
+        <collision>
+        <origin xyz="0 0 0" rpy="0 0 0"/>
+        <geometry>
+            <box size="${cam_box_size} ${cam_box_size} ${cam_box_size}"/>
+        </geometry>
+        </collision>
+        <visual>
+        <origin xyz="0 0 0" rpy="0 0 0"/>
+        <geometry>
+            <box size="${cam_box_size} ${cam_box_size} ${cam_box_size}"/>
+        </geometry>
+        <material name="red"/>
+        </visual>
+        <inertial>
+        <mass value="${cam_mass}" /> This camera was estimated from the mass(weight) of a logitech camera = 0.25kg
+        <origin xyz="0 0 0" rpy="0 0 0"/> Inertia was calculated from the inertial calculator program
+        <inertia ixx="${cam_inertia_xx}" ixy="0" ixz="0" iyy="${cam_inertia_yy}" iyz="0" izz="${cam_inertia_zz}" />
+        </inertial>
+    </link>
+    <gazebo reference="camera_link_22">
+<!--        <gravity>false</gravity>-->
+        <turnGravityOff>true</turnGravityOff>
+        <mu1>10.0</mu1>
+        <mu2>10.0</mu2>
+        <material>Gazebo/Red</material>
+        <static>true</static>
+    </gazebo>
+       <!-- Camera Link 23-->
+    <link name="camera_link_23">
+        <collision>
+        <origin xyz="0 0 0" rpy="0 0 0"/>
+        <geometry>
+            <box size="${cam_box_size} ${cam_box_size} ${cam_box_size}"/>
+        </geometry>
+        </collision>
+        <visual>
+        <origin xyz="0 0 0" rpy="0 0 0"/>
+        <geometry>
+            <box size="${cam_box_size} ${cam_box_size} ${cam_box_size}"/>
+        </geometry>
+        <material name="red"/>
+        </visual>
+        <inertial>
+        <mass value="${cam_mass}" /> This camera was estimated from the mass(weight) of a logitech camera = 0.25kg
+        <origin xyz="0 0 0" rpy="0 0 0"/> Inertia was calculated from the inertial calculator program
+        <inertia ixx="${cam_inertia_xx}" ixy="0" ixz="0" iyy="${cam_inertia_yy}" iyz="0" izz="${cam_inertia_zz}" />
+        </inertial>
+    </link>
+    <gazebo reference="camera_link_23">
+<!--        <gravity>false</gravity>-->
+        <turnGravityOff>true</turnGravityOff>
+        <mu1>10.0</mu1>
+        <mu2>10.0</mu2>
+        <material>Gazebo/Red</material>
+        <static>true</static>
+    </gazebo>
+      <!-- Camera Link 24-->
+    <link name="camera_link_24">
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